Commit message: Lock the hardware spec: DT996 servos, 34 cm, ESP32-S3 FPV
Sizes the robot around the servo actually being bought, and adds the
electronics needed to fly it from a phone. Renames the project Hexabeast.

Servo model corrected to the real part. The DT996 is an MG996R form
factor digital servo advertised at 15 kg.cm (1.49 N.m at 6 V), not the
11 kg.cm of a genuine MG996R. SERVO_TORQUE is the advertised 6 V figure
derated 25 % to 1.10 N.m: clones of this class measure nearer 11 kg.cm,
so the derating and the design margin are one number doing two jobs.
URDF effort limits follow.

tools/scale_torque.py answers how big the robot can be, extrapolating
the 0.83 N.m the Phase-1 sim measured rather than guessing. The 18
servos are a fixed 1 kg however large the frame is, so mass barely grows
while the lever arm grows linearly - torque tracks mass x reach, and
34 -> 51 cm doubles the demand for 40 % more size. Ceiling is ~41 cm
(37 with an arm); 34 cm stays comfortable even at 4.8 V. So the geometry
already simulated is the geometry to build - no change.

Arm off (ARM = False) for a plain hexapod: 18 joints, 1.32 kg, static
margin up from 52 to 73 mm without the front cantilever. The generator
handled the flag everywhere but sim.launch.py hard-coded an
arm_controller spawner, which would have failed at launch now that the
controller is absent from controllers.yaml; it reads the flag too. The
arm generator stays, dormant, so flipping the flag brings back URDF,
controllers and spawner together.

docs/bom.md is the full electronics list. Once a camera eats the GPIO
every peripheral has to share one I2C bus - two PCA9685s, the IMU, a
PCF8574 for the foot switches, an INA219 - so it leads with the address
map, verified against SERVO_CHANNELS. Notably the INA219 ships at 0x40,
colliding with the first PCA9685. Separate regulators for logic and
servos keep current spikes out of the video feed.

docs/hardware.md gains the FPV design: ESP32-S3 over the old ESP32-CAM,
SoftAP so the robot needs no router, MJPEG on /stream with a WebSocket
for control. What crosses the link is body intent - the same {vx,vy,wz}
the sim's gait node takes - never joint angles, so a dropout stops the
robot instead of putting a lossy radio inside the control loop.

Co-Authored-By: Claude Opus 5 <noreply@anthropic.com>

File: ros2_ws/src/hexapod_description/urdf/hexapod_body.urdf.xacro (robot description, xacro)
@@ -9,4 +9,5 @@
   <material name="femur"><color rgba="0.85 0.45 0.15 1"/></material>
   <material name="tibia"><color rgba="0.75 0.78 0.82 1"/></material>
+  <material name="arm"><color rgba="0.35 0.36 0.40 1"/></material>
   <link name="base_link">
     <collision><geometry><box size="0.18000 0.10000 0.02200"/></geometry></collision>
@@ -24,5 +25,5 @@
     <origin xyz="0.07500 0.05500 0.00000" rpy="0.00000 0.00000 0.78540"/>
     <axis xyz="0 0 1"/>
-    <limit lower="-1.3963" upper="1.3963" effort="0.9" velocity="6.0"/>
+    <limit lower="-1.3963" upper="1.3963" effort="1.1" velocity="6.5"/>
     <dynamics damping="0.01"/>
   </joint>
@@ -48,5 +49,5 @@
     <origin xyz="0.03000 0.00000 0.00000" rpy="0.00000 0.00000 0.00000"/>
     <axis xyz="0 -1 0"/>
-    <limit lower="-1.0123" upper="1.7802" effort="0.9" velocity="6.0"/>
+    <limit lower="-1.0123" upper="1.7802" effort="1.1" velocity="6.5"/>
     <dynamics damping="0.01"/>
   </joint>
@@ -72,5 +73,5 @@
     <origin xyz="0.06000 0.00000 0.00000" rpy="0.00000 0.00000 0.00000"/>
     <axis xyz="0 -1 0"/>
-    <limit lower="-3.0369" upper="-0.2443" effort="0.9" velocity="6.0"/>
+    <limit lower="-3.0369" upper="-0.2443" effort="1.1" velocity="6.5"/>
     <dynamics damping="0.01"/>
   </joint>
@@ -101,5 +102,5 @@
     <origin xyz="0.00000 0.07000 0.00000" rpy="0.00000 0.00000 1.57080"/>
     <axis xyz="0 0 1"/>
-    <limit lower="-1.3963" upper="1.3963" effort="0.9" velocity="6.0"/>
+    <limit lower="-1.3963" upper="1.3963" effort="1.1" velocity="6.5"/>
     <dynamics damping="0.01"/>
   </joint>
@@ -125,5 +126,5 @@
     <origin xyz="0.03000 0.00000 0.00000" rpy="0.00000 0.00000 0.00000"/>
     <axis xyz="0 -1 0"/>
-    <limit lower="-1.0123" upper="1.7802" effort="0.9" velocity="6.0"/>
+    <limit lower="-1.0123" upper="1.7802" effort="1.1" velocity="6.5"/>
     <dynamics damping="0.01"/>
   </joint>
@@ -149,5 +150,5 @@
     <origin xyz="0.06000 0.00000 0.00000" rpy="0.00000 0.00000 0.00000"/>
     <axis xyz="0 -1 0"/>
-    <limit lower="-3.0369" upper="-0.2443" effort="0.9" velocity="6.0"/>
+    <limit lower="-3.0369" upper="-0.2443" effort="1.1" velocity="6.5"/>
     <dynamics damping="0.01"/>
   </joint>
@@ -178,5 +179,5 @@
     <origin xyz="-0.07500 0.05500 0.00000" rpy="0.00000 0.00000 2.35619"/>
     <axis xyz="0 0 1"/>
-    <limit lower="-1.3963" upper="1.3963" effort="0.9" velocity="6.0"/>
+    <limit lower="-1.3963" upper="1.3963" effort="1.1" velocity="6.5"/>
     <dynamics damping="0.01"/>
   </joint>
@@ -202,5 +203,5 @@
     <origin xyz="0.03000 0.00000 0.00000" rpy="0.00000 0.00000 0.00000"/>
     <axis xyz="0 -1 0"/>
-    <limit lower="-1.0123" upper="1.7802" effort="0.9" velocity="6.0"/>
+    <limit lower="-1.0123" upper="1.7802" effort="1.1" velocity="6.5"/>
     <dynamics damping="0.01"/>
   </joint>
@@ -226,5 +227,5 @@
     <origin xyz="0.06000 0.00000 0.00000" rpy="0.00000 0.00000 0.00000"/>
     <axis xyz="0 -1 0"/>
-    <limit lower="-3.0369" upper="-0.2443" effort="0.9" velocity="6.0"/>
+    <limit lower="-3.0369" upper="-0.2443" effort="1.1" velocity="6.5"/>
     <dynamics damping="0.01"/>
   </joint>
@@ -255,5 +256,5 @@
     <origin xyz="0.07500 -0.05500 0.00000" rpy="0.00000 0.00000 -0.78540"/>
     <axis xyz="0 0 1"/>
-    <limit lower="-1.3963" upper="1.3963" effort="0.9" velocity="6.0"/>
+    <limit lower="-1.3963" upper="1.3963" effort="1.1" velocity="6.5"/>
     <dynamics damping="0.01"/>
   </joint>
@@ -279,5 +280,5 @@
     <origin xyz="0.03000 0.00000 0.00000" rpy="0.00000 0.00000 0.00000"/>
     <axis xyz="0 -1 0"/>
-    <limit lower="-1.0123" upper="1.7802" effort="0.9" velocity="6.0"/>
+    <limit lower="-1.0123" upper="1.7802" effort="1.1" velocity="6.5"/>
     <dynamics damping="0.01"/>
   </joint>
@@ -303,5 +304,5 @@
     <origin xyz="0.06000 0.00000 0.00000" rpy="0.00000 0.00000 0.00000"/>
     <axis xyz="0 -1 0"/>
-    <limit lower="-3.0369" upper="-0.2443" effort="0.9" velocity="6.0"/>
+    <limit lower="-3.0369" upper="-0.2443" effort="1.1" velocity="6.5"/>
     <dynamics damping="0.01"/>
   </joint>
@@ -332,5 +333,5 @@
     <origin xyz="0.00000 -0.07000 0.00000" rpy="0.00000 0.00000 -1.57080"/>
     <axis xyz="0 0 1"/>
-    <limit lower="-1.3963" upper="1.3963" effort="0.9" velocity="6.0"/>
+    <limit lower="-1.3963" upper="1.3963" effort="1.1" velocity="6.5"/>
     <dynamics damping="0.01"/>
   </joint>
@@ -356,5 +357,5 @@
     <origin xyz="0.03000 0.00000 0.00000" rpy="0.00000 0.00000 0.00000"/>
     <axis xyz="0 -1 0"/>
-    <limit lower="-1.0123" upper="1.7802" effort="0.9" velocity="6.0"/>
+    <limit lower="-1.0123" upper="1.7802" effort="1.1" velocity="6.5"/>
     <dynamics damping="0.01"/>
   </joint>
@@ -380,5 +381,5 @@
     <origin xyz="0.06000 0.00000 0.00000" rpy="0.00000 0.00000 0.00000"/>
     <axis xyz="0 -1 0"/>
-    <limit lower="-3.0369" upper="-0.2443" effort="0.9" velocity="6.0"/>
+    <limit lower="-3.0369" upper="-0.2443" effort="1.1" velocity="6.5"/>
     <dynamics damping="0.01"/>
   </joint>
@@ -409,5 +410,5 @@
     <origin xyz="-0.07500 -0.05500 0.00000" rpy="0.00000 0.00000 -2.35619"/>
     <axis xyz="0 0 1"/>
-    <limit lower="-1.3963" upper="1.3963" effort="0.9" velocity="6.0"/>
+    <limit lower="-1.3963" upper="1.3963" effort="1.1" velocity="6.5"/>
     <dynamics damping="0.01"/>
   </joint>
@@ -433,5 +434,5 @@
     <origin xyz="0.03000 0.00000 0.00000" rpy="0.00000 0.00000 0.00000"/>
     <axis xyz="0 -1 0"/>
-    <limit lower="-1.0123" upper="1.7802" effort="0.9" velocity="6.0"/>
+    <limit lower="-1.0123" upper="1.7802" effort="1.1" velocity="6.5"/>
     <dynamics damping="0.01"/>
   </joint>
@@ -457,5 +458,5 @@
     <origin xyz="0.06000 0.00000 0.00000" rpy="0.00000 0.00000 0.00000"/>
     <axis xyz="0 -1 0"/>
-    <limit lower="-3.0369" upper="-0.2443" effort="0.9" velocity="6.0"/>
+    <limit lower="-3.0369" upper="-0.2443" effort="1.1" velocity="6.5"/>
     <dynamics damping="0.01"/>
   </joint>
