Commit message: Scale the leg to 42 % of the CAD and keep the DT996 servos
Replaces the placeholder 30/60/90 chain with the measured CAD leg scaled
to fit the servos already chosen. Links become 25 / 59 / 109 mm, holding
the CAD's proportions to within a percent - the same leg, smaller, not a
different design. Stance reach 102 mm, foot span 344 mm, all-up 1.61 kg.
Torque 0.54 N.m standing and 0.94 N.m climbing against 1.12 usable, a
1.19x margin.

Not the 33 % originally asked for, because torque was never what blocked
it: at 33 % the margin was a comfortable 1.9x, but articulation 1 fell to
27 mm while still needing to bolt on a 40.7 mm servo. Servos are a fixed
size, so uniform scaling fails from below long before it fails on torque.
Link lengths scale; servo interfaces must be redrawn at full size.

Masses now come from the STL volumes plus real servo weights rather than
guesses, and a link carries the mass of the servo it holds, not the one
driving it. The robot is 77 % servo by weight - the reason PLA thickness
barely moves the torque budget while stance reach dominates it.

Servo centres move to 0 / 45 / -105 deg. These are horn-fitting angles
and nothing about them survives a geometry change; worst-case excursions
are coxa 44, femur 62, tibia 68 deg, inside the 80 deg of usable travel.

tools/check_ik.py had the Phase-0 geometry hardcoded and was reporting
stale calibration for the new leg. It reads robot_config now, which is
what let the centres be recomputed at all.

docs/cad-measurements.md also corrects an error in the previous commit:
scale_torque's reach is the stance lever arm, not the link chain, and
feeding it the extended chain overstated torque 1.9x. The CAD leg is
2.3x over budget, not 4.4x.

Co-Authored-By: Claude Opus 5 <noreply@anthropic.com>

File: ros2_ws/src/hexapod_description/urdf/hexapod_body.urdf.xacro (robot description, xacro)
@@ -15,6 +15,6 @@
     <inertial>
       <origin xyz="0.00000 0.00000 0.00000"/>
-      <mass value="0.45"/>
-      <inertia ixx="3.932e-04" iyy="1.233e-03" izz="1.590e-03" ixy="0" ixz="0" iyz="0"/>
+      <mass value="0.79"/>
+      <inertia ixx="6.902e-04" iyy="2.165e-03" izz="2.791e-03" ixy="0" ixz="0" iyz="0"/>
     </inertial>
   </link>
@@ -30,16 +30,16 @@
   <link name="FL_coxa_link">
     <collision>
-      <origin xyz="0.01500 0.00000 0.00000"/>
-      <geometry><box size="0.03000 0.01600 0.01600"/></geometry>
-    </collision>
-    <visual>
-      <origin xyz="0.01500 0.00000 0.00000"/>
-      <geometry><box size="0.03000 0.01600 0.01600"/></geometry>
-      <material name="coxa"/>
-    </visual>
-    <inertial>
-      <origin xyz="0.01500 0.00000 0.00000"/>
-      <mass value="0.06"/>
-      <inertia ixx="5.026e-04" iyy="5.058e-04" izz="5.058e-04" ixy="0" ixz="0" iyz="0"/>
+      <origin xyz="0.01250 0.00000 0.00000"/>
+      <geometry><box size="0.02500 0.01600 0.01600"/></geometry>
+    </collision>
+    <visual>
+      <origin xyz="0.01250 0.00000 0.00000"/>
+      <geometry><box size="0.02500 0.01600 0.01600"/></geometry>
+      <material name="coxa"/>
+    </visual>
+    <inertial>
+      <origin xyz="0.01250 0.00000 0.00000"/>
+      <mass value="0.065"/>
+      <inertia ixx="5.028e-04" iyy="5.048e-04" izz="5.048e-04" ixy="0" ixz="0" iyz="0"/>
     </inertial>
   </link>
@@ -47,23 +47,23 @@
     <parent link="FL_coxa_link"/>
     <child link="FL_femur_link"/>
-    <origin xyz="0.03000 0.00000 0.00000" rpy="0.00000 0.00000 0.00000"/>
-    <axis xyz="0 -1 0"/>
-    <limit lower="-1.0123" upper="1.7802" effort="1.1" velocity="6.5"/>
+    <origin xyz="0.02500 0.00000 0.00000" rpy="0.00000 0.00000 0.00000"/>
+    <axis xyz="0 -1 0"/>
+    <limit lower="-0.6109" upper="2.1817" effort="1.1" velocity="6.5"/>
     <dynamics damping="0.01"/>
   </joint>
   <link name="FL_femur_link">
     <collision>
-      <origin xyz="0.03000 0.00000 0.00000"/>
-      <geometry><box size="0.06000 0.01400 0.01400"/></geometry>
-    </collision>
-    <visual>
-      <origin xyz="0.03000 0.00000 0.00000"/>
-      <geometry><box size="0.06000 0.01400 0.01400"/></geometry>
-      <material name="femur"/>
-    </visual>
-    <inertial>
-      <origin xyz="0.03000 0.00000 0.00000"/>
-      <mass value="0.065"/>
-      <inertia ixx="5.021e-04" iyy="5.206e-04" izz="5.206e-04" ixy="0" ixz="0" iyz="0"/>
+      <origin xyz="0.02950 0.00000 0.00000"/>
+      <geometry><box size="0.05900 0.01400 0.01400"/></geometry>
+    </collision>
+    <visual>
+      <origin xyz="0.02950 0.00000 0.00000"/>
+      <geometry><box size="0.05900 0.01400 0.01400"/></geometry>
+      <material name="femur"/>
+    </visual>
+    <inertial>
+      <origin xyz="0.02950 0.00000 0.00000"/>
+      <mass value="0.063"/>
+      <inertia ixx="5.021e-04" iyy="5.193e-04" izz="5.193e-04" ixy="0" ixz="0" iyz="0"/>
     </inertial>
   </link>
@@ -71,27 +71,27 @@
     <parent link="FL_femur_link"/>
     <child link="FL_tibia_link"/>
-    <origin xyz="0.06000 0.00000 0.00000" rpy="0.00000 0.00000 0.00000"/>
-    <axis xyz="0 -1 0"/>
-    <limit lower="-3.0369" upper="-0.2443" effort="1.1" velocity="6.5"/>
+    <origin xyz="0.05900 0.00000 0.00000" rpy="0.00000 0.00000 0.00000"/>
+    <axis xyz="0 -1 0"/>
+    <limit lower="-3.2289" upper="-0.4363" effort="1.1" velocity="6.5"/>
     <dynamics damping="0.01"/>
   </joint>
   <link name="FL_tibia_link">
     <collision>
-      <origin xyz="0.09000 0 0"/>
-      <geometry><sphere radius="0.008"/></geometry>
-    </collision>
-    <collision>
-      <origin xyz="0.04500 0.00000 0.00000" rpy="0 1.570796 0"/>
-      <geometry><cylinder radius="0.0055" length="0.0740"/></geometry>
-    </collision>
-    <visual>
-      <origin xyz="0.04500 0.00000 0.00000"/>
-      <geometry><box size="0.09000 0.01100 0.01100"/></geometry>
-      <material name="tibia"/>
-    </visual>
-    <inertial>
-      <origin xyz="0.04500 0.00000 0.00000"/>
-      <mass value="0.02"/>
-      <inertia ixx="5.004e-04" iyy="5.137e-04" izz="5.137e-04" ixy="0" ixz="0" iyz="0"/>
+      <origin xyz="0.10900 0 0"/>
+      <geometry><sphere radius="0.008"/></geometry>
+    </collision>
+    <collision>
+      <origin xyz="0.05450 0.00000 0.00000" rpy="0 1.570796 0"/>
+      <geometry><cylinder radius="0.0055" length="0.0930"/></geometry>
+    </collision>
+    <visual>
+      <origin xyz="0.05450 0.00000 0.00000"/>
+      <geometry><box size="0.10900 0.01100 0.01100"/></geometry>
+      <material name="tibia"/>
+    </visual>
+    <inertial>
+      <origin xyz="0.05450 0.00000 0.00000"/>
+      <mass value="0.008"/>
+      <inertia ixx="5.002e-04" iyy="5.080e-04" izz="5.080e-04" ixy="0" ixz="0" iyz="0"/>
     </inertial>
   </link>
@@ -107,16 +107,16 @@
   <link name="ML_coxa_link">
     <collision>
-      <origin xyz="0.01500 0.00000 0.00000"/>
-      <geometry><box size="0.03000 0.01600 0.01600"/></geometry>
-    </collision>
-    <visual>
-      <origin xyz="0.01500 0.00000 0.00000"/>
-      <geometry><box size="0.03000 0.01600 0.01600"/></geometry>
-      <material name="coxa"/>
-    </visual>
-    <inertial>
-      <origin xyz="0.01500 0.00000 0.00000"/>
-      <mass value="0.06"/>
-      <inertia ixx="5.026e-04" iyy="5.058e-04" izz="5.058e-04" ixy="0" ixz="0" iyz="0"/>
+      <origin xyz="0.01250 0.00000 0.00000"/>
+      <geometry><box size="0.02500 0.01600 0.01600"/></geometry>
+    </collision>
+    <visual>
+      <origin xyz="0.01250 0.00000 0.00000"/>
+      <geometry><box size="0.02500 0.01600 0.01600"/></geometry>
+      <material name="coxa"/>
+    </visual>
+    <inertial>
+      <origin xyz="0.01250 0.00000 0.00000"/>
+      <mass value="0.065"/>
+      <inertia ixx="5.028e-04" iyy="5.048e-04" izz="5.048e-04" ixy="0" ixz="0" iyz="0"/>
     </inertial>
   </link>
@@ -124,23 +124,23 @@
     <parent link="ML_coxa_link"/>
     <child link="ML_femur_link"/>
-    <origin xyz="0.03000 0.00000 0.00000" rpy="0.00000 0.00000 0.00000"/>
-    <axis xyz="0 -1 0"/>
-    <limit lower="-1.0123" upper="1.7802" effort="1.1" velocity="6.5"/>
+    <origin xyz="0.02500 0.00000 0.00000" rpy="0.00000 0.00000 0.00000"/>
+    <axis xyz="0 -1 0"/>
+    <limit lower="-0.6109" upper="2.1817" effort="1.1" velocity="6.5"/>
     <dynamics damping="0.01"/>
   </joint>
   <link name="ML_femur_link">
     <collision>
-      <origin xyz="0.03000 0.00000 0.00000"/>
-      <geometry><box size="0.06000 0.01400 0.01400"/></geometry>
-    </collision>
-    <visual>
-      <origin xyz="0.03000 0.00000 0.00000"/>
-      <geometry><box size="0.06000 0.01400 0.01400"/></geometry>
-      <material name="femur"/>
-    </visual>
-    <inertial>
-      <origin xyz="0.03000 0.00000 0.00000"/>
-      <mass value="0.065"/>
-      <inertia ixx="5.021e-04" iyy="5.206e-04" izz="5.206e-04" ixy="0" ixz="0" iyz="0"/>
+      <origin xyz="0.02950 0.00000 0.00000"/>
+      <geometry><box size="0.05900 0.01400 0.01400"/></geometry>
+    </collision>
+    <visual>
+      <origin xyz="0.02950 0.00000 0.00000"/>
+      <geometry><box size="0.05900 0.01400 0.01400"/></geometry>
+      <material name="femur"/>
+    </visual>
+    <inertial>
+      <origin xyz="0.02950 0.00000 0.00000"/>
+      <mass value="0.063"/>
+      <inertia ixx="5.021e-04" iyy="5.193e-04" izz="5.193e-04" ixy="0" ixz="0" iyz="0"/>
     </inertial>
   </link>
@@ -148,27 +148,27 @@
     <parent link="ML_femur_link"/>
     <child link="ML_tibia_link"/>
-    <origin xyz="0.06000 0.00000 0.00000" rpy="0.00000 0.00000 0.00000"/>
-    <axis xyz="0 -1 0"/>
-    <limit lower="-3.0369" upper="-0.2443" effort="1.1" velocity="6.5"/>
+    <origin xyz="0.05900 0.00000 0.00000" rpy="0.00000 0.00000 0.00000"/>
+    <axis xyz="0 -1 0"/>
+    <limit lower="-3.2289" upper="-0.4363" effort="1.1" velocity="6.5"/>
     <dynamics damping="0.01"/>
   </joint>
   <link name="ML_tibia_link">
     <collision>
-      <origin xyz="0.09000 0 0"/>
-      <geometry><sphere radius="0.008"/></geometry>
-    </collision>
-    <collision>
-      <origin xyz="0.04500 0.00000 0.00000" rpy="0 1.570796 0"/>
-      <geometry><cylinder radius="0.0055" length="0.0740"/></geometry>
-    </collision>
-    <visual>
-      <origin xyz="0.04500 0.00000 0.00000"/>
-      <geometry><box size="0.09000 0.01100 0.01100"/></geometry>
-      <material name="tibia"/>
-    </visual>
-    <inertial>
-      <origin xyz="0.04500 0.00000 0.00000"/>
-      <mass value="0.02"/>
-      <inertia ixx="5.004e-04" iyy="5.137e-04" izz="5.137e-04" ixy="0" ixz="0" iyz="0"/>
+      <origin xyz="0.10900 0 0"/>
+      <geometry><sphere radius="0.008"/></geometry>
+    </collision>
+    <collision>
+      <origin xyz="0.05450 0.00000 0.00000" rpy="0 1.570796 0"/>
+      <geometry><cylinder radius="0.0055" length="0.0930"/></geometry>
+    </collision>
+    <visual>
+      <origin xyz="0.05450 0.00000 0.00000"/>
+      <geometry><box size="0.10900 0.01100 0.01100"/></geometry>
+      <material name="tibia"/>
+    </visual>
+    <inertial>
+      <origin xyz="0.05450 0.00000 0.00000"/>
+      <mass value="0.008"/>
+      <inertia ixx="5.002e-04" iyy="5.080e-04" izz="5.080e-04" ixy="0" ixz="0" iyz="0"/>
     </inertial>
   </link>
@@ -184,16 +184,16 @@
   <link name="RL_coxa_link">
     <collision>
-      <origin xyz="0.01500 0.00000 0.00000"/>
-      <geometry><box size="0.03000 0.01600 0.01600"/></geometry>
-    </collision>
-    <visual>
-      <origin xyz="0.01500 0.00000 0.00000"/>
-      <geometry><box size="0.03000 0.01600 0.01600"/></geometry>
-      <material name="coxa"/>
-    </visual>
-    <inertial>
-      <origin xyz="0.01500 0.00000 0.00000"/>
-      <mass value="0.06"/>
-      <inertia ixx="5.026e-04" iyy="5.058e-04" izz="5.058e-04" ixy="0" ixz="0" iyz="0"/>
+      <origin xyz="0.01250 0.00000 0.00000"/>
+      <geometry><box size="0.02500 0.01600 0.01600"/></geometry>
+    </collision>
+    <visual>
+      <origin xyz="0.01250 0.00000 0.00000"/>
+      <geometry><box size="0.02500 0.01600 0.01600"/></geometry>
+      <material name="coxa"/>
+    </visual>
+    <inertial>
+      <origin xyz="0.01250 0.00000 0.00000"/>
+      <mass value="0.065"/>
+      <inertia ixx="5.028e-04" iyy="5.048e-04" izz="5.048e-04" ixy="0" ixz="0" iyz="0"/>
     </inertial>
   </link>
@@ -201,23 +201,23 @@
     <parent link="RL_coxa_link"/>
     <child link="RL_femur_link"/>
-    <origin xyz="0.03000 0.00000 0.00000" rpy="0.00000 0.00000 0.00000"/>
-    <axis xyz="0 -1 0"/>
-    <limit lower="-1.0123" upper="1.7802" effort="1.1" velocity="6.5"/>
+    <origin xyz="0.02500 0.00000 0.00000" rpy="0.00000 0.00000 0.00000"/>
+    <axis xyz="0 -1 0"/>
+    <limit lower="-0.6109" upper="2.1817" effort="1.1" velocity="6.5"/>
     <dynamics damping="0.01"/>
   </joint>
   <link name="RL_femur_link">
     <collision>
-      <origin xyz="0.03000 0.00000 0.00000"/>
-      <geometry><box size="0.06000 0.01400 0.01400"/></geometry>
-    </collision>
-    <visual>
-      <origin xyz="0.03000 0.00000 0.00000"/>
-      <geometry><box size="0.06000 0.01400 0.01400"/></geometry>
-      <material name="femur"/>
-    </visual>
-    <inertial>
-      <origin xyz="0.03000 0.00000 0.00000"/>
-      <mass value="0.065"/>
-      <inertia ixx="5.021e-04" iyy="5.206e-04" izz="5.206e-04" ixy="0" ixz="0" iyz="0"/>
+      <origin xyz="0.02950 0.00000 0.00000"/>
+      <geometry><box size="0.05900 0.01400 0.01400"/></geometry>
+    </collision>
+    <visual>
+      <origin xyz="0.02950 0.00000 0.00000"/>
+      <geometry><box size="0.05900 0.01400 0.01400"/></geometry>
+      <material name="femur"/>
+    </visual>
+    <inertial>
+      <origin xyz="0.02950 0.00000 0.00000"/>
+      <mass value="0.063"/>
+      <inertia ixx="5.021e-04" iyy="5.193e-04" izz="5.193e-04" ixy="0" ixz="0" iyz="0"/>
     </inertial>
   </link>
@@ -225,27 +225,27 @@
     <parent link="RL_femur_link"/>
     <child link="RL_tibia_link"/>
-    <origin xyz="0.06000 0.00000 0.00000" rpy="0.00000 0.00000 0.00000"/>
-    <axis xyz="0 -1 0"/>
-    <limit lower="-3.0369" upper="-0.2443" effort="1.1" velocity="6.5"/>
+    <origin xyz="0.05900 0.00000 0.00000" rpy="0.00000 0.00000 0.00000"/>
+    <axis xyz="0 -1 0"/>
+    <limit lower="-3.2289" upper="-0.4363" effort="1.1" velocity="6.5"/>
     <dynamics damping="0.01"/>
   </joint>
   <link name="RL_tibia_link">
     <collision>
-      <origin xyz="0.09000 0 0"/>
-      <geometry><sphere radius="0.008"/></geometry>
-    </collision>
-    <collision>
-      <origin xyz="0.04500 0.00000 0.00000" rpy="0 1.570796 0"/>
-      <geometry><cylinder radius="0.0055" length="0.0740"/></geometry>
-    </collision>
-    <visual>
-      <origin xyz="0.04500 0.00000 0.00000"/>
-      <geometry><box size="0.09000 0.01100 0.01100"/></geometry>
-      <material name="tibia"/>
-    </visual>
-    <inertial>
-      <origin xyz="0.04500 0.00000 0.00000"/>
-      <mass value="0.02"/>
-      <inertia ixx="5.004e-04" iyy="5.137e-04" izz="5.137e-04" ixy="0" ixz="0" iyz="0"/>
+      <origin xyz="0.10900 0 0"/>
+      <geometry><sphere radius="0.008"/></geometry>
+    </collision>
+    <collision>
+      <origin xyz="0.05450 0.00000 0.00000" rpy="0 1.570796 0"/>
+      <geometry><cylinder radius="0.0055" length="0.0930"/></geometry>
+    </collision>
+    <visual>
+      <origin xyz="0.05450 0.00000 0.00000"/>
+      <geometry><box size="0.10900 0.01100 0.01100"/></geometry>
+      <material name="tibia"/>
+    </visual>
+    <inertial>
+      <origin xyz="0.05450 0.00000 0.00000"/>
+      <mass value="0.008"/>
+      <inertia ixx="5.002e-04" iyy="5.080e-04" izz="5.080e-04" ixy="0" ixz="0" iyz="0"/>
     </inertial>
   </link>
@@ -261,16 +261,16 @@
   <link name="FR_coxa_link">
     <collision>
-      <origin xyz="0.01500 0.00000 0.00000"/>
-      <geometry><box size="0.03000 0.01600 0.01600"/></geometry>
-    </collision>
-    <visual>
-      <origin xyz="0.01500 0.00000 0.00000"/>
-      <geometry><box size="0.03000 0.01600 0.01600"/></geometry>
-      <material name="coxa"/>
-    </visual>
-    <inertial>
-      <origin xyz="0.01500 0.00000 0.00000"/>
-      <mass value="0.06"/>
-      <inertia ixx="5.026e-04" iyy="5.058e-04" izz="5.058e-04" ixy="0" ixz="0" iyz="0"/>
+      <origin xyz="0.01250 0.00000 0.00000"/>
+      <geometry><box size="0.02500 0.01600 0.01600"/></geometry>
+    </collision>
+    <visual>
+      <origin xyz="0.01250 0.00000 0.00000"/>
+      <geometry><box size="0.02500 0.01600 0.01600"/></geometry>
+      <material name="coxa"/>
+    </visual>
+    <inertial>
+      <origin xyz="0.01250 0.00000 0.00000"/>
+      <mass value="0.065"/>
+      <inertia ixx="5.028e-04" iyy="5.048e-04" izz="5.048e-04" ixy="0" ixz="0" iyz="0"/>
     </inertial>
   </link>
@@ -278,23 +278,23 @@
     <parent link="FR_coxa_link"/>
     <child link="FR_femur_link"/>
-    <origin xyz="0.03000 0.00000 0.00000" rpy="0.00000 0.00000 0.00000"/>
-    <axis xyz="0 -1 0"/>
-    <limit lower="-1.0123" upper="1.7802" effort="1.1" velocity="6.5"/>
+    <origin xyz="0.02500 0.00000 0.00000" rpy="0.00000 0.00000 0.00000"/>
+    <axis xyz="0 -1 0"/>
+    <limit lower="-0.6109" upper="2.1817" effort="1.1" velocity="6.5"/>
     <dynamics damping="0.01"/>
   </joint>
   <link name="FR_femur_link">
     <collision>
-      <origin xyz="0.03000 0.00000 0.00000"/>
-      <geometry><box size="0.06000 0.01400 0.01400"/></geometry>
-    </collision>
-    <visual>
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
File: ros2_ws/src/hexapod_description/urdf/hexapod_control.xacro (robot description, xacro)
@@ -13,10 +13,10 @@
     <joint name="FL_femur">
       <command_interface name="position"/>
-      <state_interface name="position"><param name="initial_value">0.3840</param></state_interface>
+      <state_interface name="position"><param name="initial_value">0.7854</param></state_interface>
       <state_interface name="velocity"/>
     </joint>
     <joint name="FL_tibia">
       <command_interface name="position"/>
-      <state_interface name="position"><param name="initial_value">-1.6406</param></state_interface>
+      <state_interface name="position"><param name="initial_value">-1.8326</param></state_interface>
       <state_interface name="velocity"/>
     </joint>
@@ -28,10 +28,10 @@
     <joint name="ML_femur">
       <command_interface name="position"/>
-      <state_interface name="position"><param name="initial_value">0.3840</param></state_interface>
+      <state_interface name="position"><param name="initial_value">0.7854</param></state_interface>
       <state_interface name="velocity"/>
     </joint>
     <joint name="ML_tibia">
       <command_interface name="position"/>
-      <state_interface name="position"><param name="initial_value">-1.6406</param></state_interface>
+      <state_interface name="position"><param name="initial_value">-1.8326</param></state_interface>
       <state_interface name="velocity"/>
     </joint>
@@ -43,10 +43,10 @@
     <joint name="RL_femur">
       <command_interface name="position"/>
-      <state_interface name="position"><param name="initial_value">0.3840</param></state_interface>
+      <state_interface name="position"><param name="initial_value">0.7854</param></state_interface>
       <state_interface name="velocity"/>
     </joint>
     <joint name="RL_tibia">
       <command_interface name="position"/>
-      <state_interface name="position"><param name="initial_value">-1.6406</param></state_interface>
+      <state_interface name="position"><param name="initial_value">-1.8326</param></state_interface>
       <state_interface name="velocity"/>
     </joint>
@@ -58,10 +58,10 @@
     <joint name="FR_femur">
       <command_interface name="position"/>
-      <state_interface name="position"><param name="initial_value">0.3840</param></state_interface>
+      <state_interface name="position"><param name="initial_value">0.7854</param></state_interface>
       <state_interface name="velocity"/>
     </joint>
     <joint name="FR_tibia">
       <command_interface name="position"/>
-      <state_interface name="position"><param name="initial_value">-1.6406</param></state_interface>
+      <state_interface name="position"><param name="initial_value">-1.8326</param></state_interface>
       <state_interface name="velocity"/>
     </joint>
@@ -73,10 +73,10 @@
     <joint name="MR_femur">
       <command_interface name="position"/>
-      <state_interface name="position"><param name="initial_value">0.3840</param></state_interface>
+      <state_interface name="position"><param name="initial_value">0.7854</param></state_interface>
       <state_interface name="velocity"/>
     </joint>
     <joint name="MR_tibia">
       <command_interface name="position"/>
-      <state_interface name="position"><param name="initial_value">-1.6406</param></state_interface>
+      <state_interface name="position"><param name="initial_value">-1.8326</param></state_interface>
       <state_interface name="velocity"/>
     </joint>
@@ -88,10 +88,10 @@
     <joint name="RR_femur">
       <command_interface name="position"/>
-      <state_interface name="position"><param name="initial_value">0.3840</param></state_interface>
+      <state_interface name="position"><param name="initial_value">0.7854</param></state_interface>
       <state_interface name="velocity"/>
     </joint>
     <joint name="RR_tibia">
       <command_interface name="position"/>
-      <state_interface name="position"><param name="initial_value">-1.6406</param></state_interface>
+      <state_interface name="position"><param name="initial_value">-1.8326</param></state_interface>
       <state_interface name="velocity"/>
     </joint>
