Commit message: Generate the whole robot: body, camera mast, stance assembly
Adds everything the legs bolt to. The body plate carries six coxa servo
mounts at the hip positions from robot_config, holes for two PCA9685s
and the ESP32-S3 carrier, battery strap slots and a socket for the mast.
The mast stands the camera above the robot, tilted 15 deg down.

The assembly is not decoration: it chains the REAL mechanical offsets -
wall thicknesses, servo heights, horn faces - and then asks where each
foot actually lands. Two findings came out of it that no render would
have shown.

Camera height is set by the knees, not the body. A front leg's knee
rises to 80 mm above the plate at the top of its swing; the first draft
put the camera at 62 mm, so the legs would have swept through the shot
every stride. The mast is 105 mm and thicker to match.

Each foot lands 11.9 mm off the ideal, identically on all six legs. The
femur servo bolts to a wall, so its shaft cannot sit on the leg's centre
plane, and the offset is exactly servo half-width + clearance + half
wall. Seen from the coxa axis this is a rotation rather than a reach
error: the stance hexagon is turned 6.65 deg and the true radius is
102.69 against a nominal 102. Trimming each coxa by -6.65 deg returns
the feet to the model's radial line for 0.7 mm of residual - under 1 %,
so torque and gait are unaffected. All six legs are offset the same
rotational sense, which keeps the stance symmetric AND keeps all six
legs one printed part rather than mirrored pairs.

An earlier version of the check also reported a 22 mm vertical error.
That was the check's own fault: the kinematic origin is the FEMUR AXIS
plane, where the leg's vertical motion starts, not the body plate.

MASS_BODY is now measured rather than guessed - 737 g including the
generated plate and mast - which puts the robot at 1.55 kg all-up, 0.91
N.m climbing against 1.12 usable, a 1.23x margin. URDF and the firmware
header regenerated; the firmware's 2615 checks still pass.

Co-Authored-By: Claude Opus 5 <noreply@anthropic.com>

File: ros2_ws/src/hexapod_description/urdf/hexapod_body.urdf.xacro (robot description, xacro)
@@ -15,6 +15,6 @@
     <inertial>
       <origin xyz="0.00000 0.00000 0.00000"/>
-      <mass value="0.79"/>
-      <inertia ixx="6.902e-04" iyy="2.165e-03" izz="2.791e-03" ixy="0" ixz="0" iyz="0"/>
+      <mass value="0.737"/>
+      <inertia ixx="6.439e-04" iyy="2.020e-03" izz="2.604e-03" ixy="0" ixz="0" iyz="0"/>
     </inertial>
   </link>
